File: jlink_to_mini.sch (EAGLE design)
At the start: 2 parts, among them CON1 JTAG-20_DEVICE, P1 STLINKV3_STDC14

Commit message: Added TME partnumbers
Parts:
- P1: OC_TME (none) -> ZL322-2X7P
Changed lines of the file:
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@@
 <?xml version="1.0" encoding="utf-8"?>
 <!DOCTYPE eagle SYSTEM "eagle.dtd">
-<eagle version="9.3.2">
+<eagle version="9.6.2">
 <drawing>
 <settings>
@@
 <parts>
 <part name="CON1" library="jtag" deviceset="JTAG-20_DEVICE" device=""/>
-<part name="P1" library="jtag" deviceset="STLINKV3_STDC14" device=""/>
+<part name="P1" library="jtag" deviceset="STLINKV3_STDC14" device="">
+<attribute name="OC_TME" value="ZL322-2X7P "/>
+</part>
 <part name="GND1" library="supply1" deviceset="GND" device=""/>
 <part name="GND2" library="supply1" deviceset="GND" device=""/>
@@
 <attribute name="VALUE" x="151.13" y="83.82" size="1.778" layer="96"/>
 <attribute name="NAME" x="151.13" y="107.442" size="1.778" layer="95"/>
+<attribute name="OC_TME" x="154.94" y="96.52" size="1.778" layer="96" display="off"/>
 </instance>
 <instance part="GND1" gate="1" x="106.68" y="78.74" smashed="yes">
